Commit message: diff_drive_controller

File: webots_turtlebot3_examples/urdf/turtlebot.xacro (robot description, xacro)
@@ -1,265 +1,184 @@
-<?xml version="1.0"?>
-<robot name="" xmlns:xacro="http://ros.org/wiki/xacro">
+<?xml version="1.0" ?>
+<robot name="tb3_burger_converted" xmlns:xacro="http://ros.org/wiki/xacro">
+  <!-- Init colour -->
+  <material name="black">
+      <color rgba="0.0 0.0 0.0 1.0"/>
+  </material>
+  <material name="dark">
+    <color rgba="0.3 0.3 0.3 1.0"/>
+  </material>
+  <material name="light_black">
+    <color rgba="0.4 0.4 0.4 1.0"/>
+  </material>
+  <material name="blue">
+    <color rgba="0.0 0.0 0.8 1.0"/>
+  </material>
+  <material name="green">
+    <color rgba="0.0 0.8 0.0 1.0"/>
+  </material>
+  <material name="grey">
+    <color rgba="0.5 0.5 0.5 1.0"/>
+  </material>
+  <material name="orange">
+    <color rgba="${255/255} ${108/255} ${10/255} 1.0"/>
+  </material>
+  <material name="brown">
+    <color rgba="${222/255} ${207/255} ${195/255} 1.0"/>
+  </material>
+  <material name="red">
+    <color rgba="0.8 0.0 0.0 1.0"/>
+  </material>
+  <material name="white">
+    <color rgba="1.0 1.0 1.0 1.0"/>
+  </material>
+  <link name="base_footprint"/>
+  <joint name="base_joint" type="fixed">
+    <parent link="base_footprint"/>
+    <child link="base_link"/>
+    <origin xyz="0.0 0.0 0.010" rpy="0 0 0"/>
+  </joint>
   <link name="base_link">
     <visual>
-      <origin xyz="-0.032 0 0.08" rpy="0 0 0"/>
+      <origin xyz="-0.032 0 0.0" rpy="0 0 0"/>
       <geometry>
-        <box size="0.097 0.137 0.1425"/>
+        <mesh filename="package://webots_turtlebot3_examples/meshes/burger_base_scaled.stl"/>
       </geometry>
+      <material name="light_black"/>
     </visual>
     <collision>
-      <origin xyz="-0.032 0 0.08" rpy="0 0 0"/>
+      <origin xyz="-0.032 0 0.070" rpy="0 0 0"/>
       <geometry>
-        <box size="0.097 0.137 0.1425"/>
+        <box size="0.140 0.140 0.143"/>
       </geometry>
     </collision>
-    <visual>
-      <origin xyz="-0.032 0 0.08" rpy="0 0 0"/>
+    <inertial>
+      <origin xyz="0 0 0" rpy="0 0 0"/>
+      <mass value="8.2573504e-01"/>
+      <inertia ixx="2.2124416e-03" ixy="-1.2294101e-05" ixz="3.4938785e-05"
+               iyy="2.1193702e-03" iyz="-5.0120904e-06"
+               izz="2.0064271e-03" />
+    </inertial>
+  </link>
+  <joint name="wheel_left_joint" type="continuous">
+    <parent link="base_link"/>
+    <child link="wheel_left_link"/>
+    <origin xyz="0.0 0.08 0.023" rpy="-1.57 0 0"/>
+    <axis xyz="0 0 1"/>
+  </joint>
+  <link name= "base_camera">
+    <collision>
+      <origin xyz="0.0 0.0 0.0" rpy="0 0 0"/>
       <geometry>
-        <box size="0.135 0.095 0.143"/>
-      </geometry>
-    </visual>
-    <collision>
-      <origin xyz="-0.032 0 0.08" rpy="0 0 0"/>
-      <geometry>
-        <box size="0.135 0.095 0.143"/>
+        <cylinder length="0.018" radius="0.033"/>
       </geometry>
     </collision>
   </link>
-  <link name="compass">
-  </link>
-  <joint name="base_link_compass_joint" type="fixed">
+  <joint name="base_camera_joint" type="fixed">
+    <origin xyz="-0.032 0 0.172" rpy="0 0 0"/>
     <parent link="base_link"/>
-    <child link="compass"/>
-    <origin xyz="-0.032 0 0.078" rpy="0 0 0"/>
+    <child link="base_camera"/>
   </joint>
-  <link name="gyro">
-  </link>
-  <joint name="base_link_gyro_joint" type="fixed">
-    <parent link="base_link"/>
-    <child link="gyro"/>
-    <origin xyz="-0.032 0 0.078" rpy="0 0 0"/>
-  </joint>
-  <link name="accelerometer">
-  </link>
-  <joint name="base_link_accelerometer_joint" type="fixed">
-    <parent link="base_link"/>
-    <child link="accelerometer"/>
-    <origin xyz="-0.032 0 0.078" rpy="0 0 0"/>
-  </joint>
-  <joint name="left wheel motor" type="continuous">
-    <parent link="base_link"/>
-    <child link="left wheel"/>
-    <axis xyz="-0.000003 -1 0.000003"/>
-    <limit effort="10" velocity="6.67"/>
-    <origin xyz="0 0.08 0.033" rpy="-0.526852 -1.57079 -2.614737"/>
-  </joint>
-  <link name="left wheel">
+  <link name="wheel_left_link">
     <visual>
-      <origin xyz="0 0 0" rpy="-1.570796 0 0"/>
+      <origin xyz="0 0 0" rpy="1.57 0 0"/>
       <geometry>
-        <cylinder radius="0.033" length="0.018"/>
+        <mesh filename="package://webots_turtlebot3_examples/meshes/left_tire_converted.stl"/>
       </geometry>
-    </visual>
-    <collision>
-      <origin xyz="0 0 0" rpy="-1.570796 0 0"/>
-      <geometry>
-        <cylinder radius="0.033" length="0.018"/>
-      </geometry>
-    </collision>
-  </link>
-  <joint name="right wheel motor" type="continuous">
-    <parent link="base_link"/>
-    <child link="right wheel"/>
-    <axis xyz="0 1 0"/>
-    <limit effort="10" velocity="6.67"/>
-    <origin xyz="0 -0.08 0.033" rpy="0 -1.570796 0"/>
-  </joint>
-  <link name="right wheel">
-    <visual>
-      <origin xyz="0 0 0" rpy="-1.570796 0 0"/>
-      <geometry>
-        <cylinder radius="0.033" length="0.018"/>
-      </geometry>
-    </visual>
-    <collision>
-      <origin xyz="0 0 0" rpy="-1.570796 0 0"/>
-      <geometry>
-        <cylinder radius="0.033" length="0.018"/>
-      </geometry>
-    </collision>
-  </link>
-  <link name="LDS-01">
-    <visual>
-      <origin xyz="0.014 0 -0.014" rpy="1.5708 0.00001 -1.5708"/>
-      <geometry>
-        <box size="0.07 0.01 0.1"/>
-      </geometry>
-    </visual>
-    <collision>
-      <origin xyz="0.014 0 -0.014" rpy="1.5708 0.00001 -1.5708"/>
-      <geometry>
-        <box size="0.07 0.01 0.1"/>
-      </geometry>
-    </collision>
-    <visual>
-      <origin xyz="0 0 0" rpy="0 0 0"/>
-      <geometry>
-        <cylinder radius="0.032" length="0.021"/>
-      </geometry>
+      <material name="dark"/>
     </visual>
     <collision>
       <origin xyz="0 0 0" rpy="0 0 0"/>
       <geometry>
-        <cylinder radius="0.032" length="0.021"/>
+        <cylinder length="0.018" radius="0.033"/>
       </geometry>
     </collision>
+    <inertial>
+      <origin xyz="0 0 0" />
+      <mass value="2.8498940e-02" />
+      <inertia ixx="1.1175580e-05" ixy="-4.2369783e-11" ixz="-5.9381719e-09"
+               iyy="1.1192413e-05" iyz="-1.4400107e-11"
+               izz="2.0712558e-05" />
+      </inertial>
   </link>
-  <joint name="base_link_LDS-01_joint" type="fixed">
+  <joint name="wheel_right_joint" type="continuous">
     <parent link="base_link"/>
-    <child link="LDS-01"/>
-    <origin xyz="-0.03 0 0.173" rpy="0 0 0"/>
+    <child link="wheel_right_link"/>
+    <origin xyz="0.0 -0.080 0.023" rpy="-1.57 0 0"/>
+    <axis xyz="0 0 1"/>
   </joint>
-  <link name="screw3">
+  <link name="wheel_right_link">
     <visual>
-      <origin xyz="0.01 0 0" rpy="3.141593 1.570793 3.141593"/>
+      <origin xyz="0 0 0" rpy="1.57 0 0"/>
       <geometry>
-        <cylinder radius="0.0015" length="0.02"/>
+        <mesh filename="package://webots_turtlebot3_examples/meshes/right_tire_converted.stl"/>
       </geometry>
+      <material name="dark"/>
     </visual>
     <collision>
-      <origin xyz="0.01 0 0" rpy="3.141593 1.570793 3.141593"/>
+      <origin xyz="0 0 0" rpy="0 0 0"/>
       <geometry>
-        <cylinder radius="0.0015" length="0.02"/>
+        <cylinder length="0.018" radius="0.033"/>
       </geometry>
     </collision>
+    <inertial>
+      <origin xyz="0 0 0" />
+      <mass value="2.8498940e-02" />
+      <inertia ixx="1.1175580e-05" ixy="-4.2369783e-11" ixz="-5.9381719e-09"
+               iyy="1.1192413e-05" iyz="-1.4400107e-11"
+               izz="2.0712558e-05" />
+      </inertial>
+  </link>
+  <joint name="caster_back_joint" type="fixed">
+    <parent link="base_link"/>
+    <child link="caster_back_link"/>
+    <origin xyz="-0.081 0 -0.004" rpy="-1.57 0 0"/>
+  </joint>
+  <link name="caster_back_link">
+    <collision>
+      <origin xyz="0 0.001 0" rpy="0 0 0"/>
+      <geometry>
+        <box size="0.030 0.009 0.020"/>
+      </geometry>
+    </collision>
+    <inertial>
+      <origin xyz="0 0 0" />
+      <mass value="0.005" />
+      <inertia ixx="0.001" ixy="0.0" ixz="0.0"
+               iyy="0.001" iyz="0.0"
+               izz="0.001" />
+    </inertial>
+  </link>
+  <joint name="imu_joint" type="fixed">
+    <parent link="base_link"/>
+    <child link="imu_link"/>
+    <origin xyz="-0.032 0 0.068" rpy="0 0 0"/>
+  </joint>
+  <link name="imu_link"/>
+  <joint name="scan_joint" type="fixed">
+    <parent link="base_link"/>
+    <child link="base_scan"/>
+    <origin xyz="-0.032 0 0.172" rpy="0 0 0"/>
+  </joint>
+  <link name="base_scan">
     <visual>
-      <origin xyz="-0.0015 0 0" rpy="3.141593 1.570793 3.141593"/>
+      <origin xyz="0 0 0.0" rpy="0 0 0"/>
       <geometry>
-        <cylinder radius="0.0025" length="0.003"/>
+        <mesh filename="package://webots_turtlebot3_examples/meshes/lds_converted.stl"/>
       </geometry>
+      <material name="dark"/>
     </visual>
     <collision>
-      <origin xyz="-0.0015 0 0" rpy="3.141593 1.570793 3.141593"/>
+      <origin xyz="0.015 0 -0.0065" rpy="0 0 0"/>
       <geometry>
-        <cylinder radius="0.0025" length="0.003"/>
+        <cylinder length="0.0315" radius="0.055"/>
       </geometry>
     </collision>
-  </link>
-  <joint name="LDS-01_screw3_joint" type="fixed">
-    <parent link="LDS-01"/>
-    <child link="screw3"/>
-    <origin xyz="0.035 0.0245 -0.0105" rpy="0 1.570787 0"/>
-  </joint>
-  <link name="screw2">
-    <visual>
-      <origin xyz="0.01 0 0" rpy="3.141593 1.570793 3.141593"/>
-      <geometry>
-        <cylinder radius="0.0015" length="0.02"/>
-      </geometry>
-    </visual>
-    <collision>
-      <origin xyz="0.01 0 0" rpy="3.141593 1.570793 3.141593"/>
-      <geometry>
-        <cylinder radius="0.0015" length="0.02"/>
-      </geometry>
-    </collision>
-    <visual>
-      <origin xyz="-0.0015 0 0" rpy="3.141593 1.570793 3.141593"/>
-      <geometry>
-        <cylinder radius="0.0025" length="0.003"/>
-      </geometry>
-    </visual>
-    <collision>
-      <origin xyz="-0.0015 0 0" rpy="3.141593 1.570793 3.141593"/>
-      <geometry>
-        <cylinder radius="0.0025" length="0.003"/>
-      </geometry>
-    </collision>
-  </link>
-  <joint name="LDS-01_screw2_joint" type="fixed">
-    <parent link="LDS-01"/>
-    <child link="screw2"/>
-    <origin xyz="0.035 0.0245 -0.0105" rpy="0 1.570787 0"/>
-  </joint>
-  <link name="screw1">
-    <visual>
-      <origin xyz="0.01 0 0" rpy="3.141593 1.570793 3.141593"/>
-      <geometry>
-        <cylinder radius="0.0015" length="0.02"/>
-      </geometry>
-    </visual>
-    <collision>
-      <origin xyz="0.01 0 0" rpy="3.141593 1.570793 3.141593"/>
-      <geometry>
-        <cylinder radius="0.0015" length="0.02"/>
-      </geometry>
-    </collision>
-    <visual>
-      <origin xyz="-0.0015 0 0" rpy="3.141593 1.570793 3.141593"/>
-      <geometry>
-        <cylinder radius="0.0025" length="0.003"/>
-      </geometry>
-    </visual>
-    <collision>
-      <origin xyz="-0.0015 0 0" rpy="3.141593 1.570793 3.141593"/>
-      <geometry>
-        <cylinder radius="0.0025" length="0.003"/>
-      </geometry>
-    </collision>
-  </link>
-  <joint name="LDS-01_screw1_joint" type="fixed">
-    <parent link="LDS-01"/>
-    <child link="screw1"/>
-    <origin xyz="0.035 0.0245 -0.0105" rpy="0 1.570787 0"/>
-  </joint>
-  <link name="screw0">
-    <visual>
-      <origin xyz="0.01 0 0" rpy="3.141593 1.570793 3.141593"/>
-      <geometry>
-        <cylinder radius="0.0015" length="0.02"/>
-      </geometry>
-    </visual>
-    <collision>
-      <origin xyz="0.01 0 0" rpy="3.141593 1.570793 3.141593"/>
-      <geometry>
-        <cylinder radius="0.0015" length="0.02"/>
-      </geometry>
-    </collision>
-    <visual>
-      <origin xyz="-0.0015 0 0" rpy="3.141593 1.570793 3.141593"/>
-      <geometry>
-        <cylinder radius="0.0025" length="0.003"/>
-      </geometry>
-    </visual>
-    <collision>
-      <origin xyz="-0.0015 0 0" rpy="3.141593 1.570793 3.141593"/>
-      <geometry>
-        <cylinder radius="0.0025" length="0.003"/>
-      </geometry>
-    </collision>
-  </link>
-  <joint name="LDS-01_screw0_joint" type="fixed">
-    <parent link="LDS-01"/>
-    <child link="screw0"/>
-    <origin xyz="0.035 0.0245 -0.0105" rpy="0 1.570787 0"/>
-  </joint>
-  <joint name="LDS-01_secondary_motor" type="continuous">
-    <parent link="LDS-01"/>
-    <child link="solid"/>
-    <axis xyz="0 -0.000004 1"/>
-    <limit effort="10" velocity="150"/>
-    <origin xyz="-0.046 0.01 -0.01" rpy="-0.000014 0.000005 3.141587"/>
-  </joint>
-  <link name="solid">
-  </link>
-  <joint name="LDS-01_main_motor" type="continuous">
-    <parent link="LDS-01"/>
-    <child link="solid(1)"/>
-    <axis xyz="0 -0.000004 1"/>
-    <limit effort="10" velocity="40"/>
-    <origin xyz="-0.046 0.02 -0.01" rpy="-0.000014 0.000005 3.141587"/>
-  </joint>
-  <link name="solid(1)">
+    <inertial>
+      <mass value="0.114" />
+      <origin xyz="0 0 0" />
+      <inertia ixx="0.001" ixy="0.0" ixz="0.0"
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